File: sht4x-mikrobus/sht4x-mikrobus.kicad_sch (KiCad schematic)
At the start: 8 parts, among them J1 MikroBus Left, J2 MikroBus Right, U1 SHT4x

Commit message: Refresh schematic with KiCad 10 - Use custom symbol for the Mikrobus connectors - Removed extra C2 capacitor which wasn't really needed - Jumper was the wrong way round - Added titles to sheet
Parts:
- removed C2: 4.7uF, Capacitor_SMD:C_0603_1608Metric, symbol Device:C_Small
- removed JP1: SolderJumper_3_Open, Jumper:SolderJumper-3_P1.3mm_Bridged123_Pad1.0x1.5mm, symbol Jumper:SolderJumper_3_Open
- added JP1: I2C Pullup, Jumper:SolderJumper-3_P1.3mm_Bridged123_Pad1.0x1.5mm, symbol Jumper:SolderJumper_3_Bridged123
- C1: footprint Capacitor_SMD:C_0603_1608Metric -> Capacitor_SMD:C_0402_1005Metric; LCSC C14663 -> C1525
- J1: value MikroBus Left -> Mikrobus Left; symbol Connector_Generic:Conn_01x08 -> Mikrobus:Mikrobus_AddOn_Left
- J2: value MikroBus Right -> Mikrobus Right; symbol Connector_Generic:Conn_01x08 -> Mikrobus:Mikrobus_AddOn_Right
Connections:
- net +3.3V: now also JP1.2 (C)
- net at R2.1: now also JP1.3 (B)
- net at R1.1: now also JP1.1 (A)
- no-connect marks 0 -> 11
Other:
- company: (none) -> aelius labs
- title: (none) -> SHT4X Mikrobus Module
