File: modbus-th-sensor.kicad_sch (KiCad schematic)
At the start: 41 parts, among them J1 Screw Terminal, J2 FTDI Serial, J3 ICSP, Q1 AO3401A, SW2 TERM, SW3 Node ID, U1 ATmega328P-A, U2 SHT4x, U3 SP3485EN, U5 AP63203WU, Y1 8MHz

Commit message: Updated symbols in KiCad 10. Replaced SHT4x with header for seperate sensor board
Parts:
- removed C15: 0.1uF, Capacitor_SMD:C_0402_1005Metric, symbol Device:C_Small
- removed R4, R5: 4.7k, Resistor_SMD:R_0603_1608Metric, symbol Device:R_Small
- removed U2: SHT4x, Sensor_Humidity:Sensirion_DFN-4_1.5x1.5mm_P0.8mm_SHT4x_NoCentralPad, symbol Sensor_Humidity:SHT4x
- added J4: Sensor, Connector_PinSocket_2.54mm:PinSocket_1x05_P2.54mm_Horizontal, symbol Connector:Conn_01x05_Socket
Connections:
- net +3.3V: now also J4.1 (Pin_1)
- net GND: now also J4.5 (Pin_5)
- net SCL: now also J4.3 (Pin_3)
- net SDA: now also J4.2 (Pin_2)
- net INT: now reaches U1.26 (PC3)
- net INT: now also J4.4 (Pin_4)
- no-connect marks 9 -> 8

Commit message: Replaced SP3485 with THVD2410, which has built-in protection
Parts:
- removed D4: SM712, Package_TO_SOT_SMD:SOT-23, symbol Diode:SM712_SOT23
- U3: value SP3485EN -> THVD2410DR; LCSC C8963 -> C1849398
Other:
- moved on the sheet: C14, R6, SW2, U3

Commit message: Added Qwiic connector
Parts:
- added J5: Qwiic, Connector_JST:JST_SH_SM04B-SRSS-TB_1x04-1MP_P1.00mm_Horizontal, symbol Connector_Generic:Conn_01x04
- J4: value Sensor -> Sensor Board
Connections:
- net +3.3V: now also J5.2 (Pin_2)
- net GND: now also J5.1 (Pin_1)
- net SCL: now also J5.4 (Pin_4)
- net SDA: now also J5.3 (Pin_3)
Other:
- moved on the sheet: J4

Commit message: Rework power input for 5-24V and fix part/footprint mismatches - Change TVS D1 from SMAJ18CA to SMAJ24CA (C148223); the SMAJ18CA   starts conducting at 20V, below the new 24V maximum input - Replace buck inductor with a shielded Sunlord SWPA4030S4R7MT 4.7uH (C57269) - Change C1 value from 47uF to 22uF to match its LCSC part (C336302) - Change C5/C6 footprints from 0603 to 0805 to match C45783 - Change F1 footprint from 1206 to 1812 to match C151170 - Update input voltage note from "5V - 15V" to "5V - 24V"
Parts:
- removed D1: SMAJ18CA, Diode_SMD:D_SMA, symbol Diode:SMAJ18CA
- added D1: SMAJ24CA, Diode_SMD:D_SMA, symbol Diode:SMAJ24CA
- C1: value 47uF -> 22uF
- C5, C6: footprint Capacitor_SMD:C_0603_1608Metric -> Capacitor_SMD:C_0805_2012Metric
- F1: footprint Fuse:Fuse_1206_3216Metric -> Fuse:Fuse_1812_4532Metric
- L1: renamed from L2; footprint Inductor_SMD:L_1812_4532Metric -> Inductor_SMD:L_Sunlord_SWPA4030S; LCSC C394127 -> C57269
- R1: value 100K -> 470K; LCSC C25803 -> C23178
Connections:
- net GND: now also D1.1 (A1)
- net at F1.2, Q1.3 (D): now also D1.2 (A2)
Other:
- note added: "5V - 24V Input Voltage"
- note removed: "5V - 15V Input Voltage"
Changed lines of the file:
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@@
 		)
 	)
-	(text "5V - 15V\nInput Voltage\n"
+	(text "5V - 24V\nInput Voltage\n"
 		(exclude_from_sim no)
 		(at 62.992 31.496 0)
@@
 		(dnp no)
 		(fields_autoplaced yes)
-		(property "Reference" "L2"
+		(property "Reference" "L1"
 			(at 190.5 26.67 90)
 			(show_name no)
@@
 			)
 		)
-		(property "Footprint" "Inductor_SMD:L_1812_4532Metric"
+		(property "Footprint" "Inductor_SMD:L_Sunlord_SWPA4030S"
 			(at 190.5 31.75 0)
 			(hide yes)
@@
 			)
 		)
-		(property "LCSC" "C394127"
+		(property "LCSC" "C57269"
 			(at 190.5 31.75 0)
 			(hide yes)
@@
 			(project "modbus-th-sensor"
 				(path "/0ebab830-f561-40b5-8ce2-2e04f313e8a8"
-					(reference "L2")
+					(reference "L1")
 					(unit 1)
 				)
@@
 			)
 		)
-		(property "Footprint" "Fuse:Fuse_1206_3216Metric"
+		(property "Footprint" "Fuse:Fuse_1812_4532Metric"
 			(at 86.36 30.48 0)
 			(hide yes)
@@
 			)
 		)
-		(property "Footprint" "Capacitor_SMD:C_0603_1608Metric"
+		(property "Footprint" "Capacitor_SMD:C_0805_2012Metric"
 			(at 212.09 43.18 0)
 			(hide yes)
@@
 	)
 	(symbol
-		(lib_id "Diode:SMAJ18CA")
-		(at 86.36 40.64 90)
-		(unit 1)
-		(body_style 1)
-		(exclude_from_sim no)
-		(in_bom yes)
-		(on_board yes)
-		(in_pos_files yes)
-		(dnp no)
-		(fields_autoplaced yes)
-		(property "Reference" "D1"
-			(at 88.9 39.3699 90)
-			(show_name no)
-			(do_not_autoplace no)
-			(effects
-				(font
-					(size 1.27 1.27)
-				)
-				(justify right)
-			)
-		)
-		(property "Value" "SMAJ18CA"
-			(at 88.9 41.9099 90)
-			(show_name no)
-			(do_not_autoplace no)
-			(effects
-				(font
-					(size 1.27 1.27)
-				)
-				(justify right)
-			)
-		)
-		(property "Footprint" "Diode_SMD:D_SMA"
-			(at 91.44 40.64 0)
-			(hide yes)
-			(show_name no)
-			(do_not_autoplace no)
-			(effects
-				(font
-					(size 1.27 1.27)
-				)
-			)
-		)
-		(property "Datasheet" "https://www.littelfuse.com/media?resourcetype=datasheets&itemid=75e32973-b177-4ee3-a0ff-cedaf1abdb93&filename=smaj-datasheet"
-			(at 86.36 40.64 0)
-			(hide yes)
-			(show_name no)
-			(do_not_autoplace no)
-			(effects
-				(font
-					(size 1.27 1.27)
-				)
-			)
-		)
-		(property "Description" "400W bidirectional Transient Voltage Suppressor, 18.0Vr, SMA(DO-214AC)"
-			(at 86.36 40.64 0)
-			(hide yes)
-			(show_name no)
-			(do_not_autoplace no)
-			(effects
-				(font
-					(size 1.27 1.27)
-				)
-			)
-		)
-		(property "LCSC" "C151240"
-			(at 86.36 40.64 90)
-			(hide yes)
-			(show_name no)
-			(do_not_autoplace no)
-			(effects
-				(font
-					(size 1.27 1.27)
-				)
-			)
-		)
-		(pin "2"
-		)
-		(pin "1"
-		)
-		(instances
-			(project "modbus-th-sensor"
-				(path "/0ebab830-f561-40b5-8ce2-2e04f313e8a8"
-					(reference "D1")
-					(unit 1)
-				)
-			)
-		)
-	)
-	(symbol
 		(lib_id "power:GND")
 		(at 57.15 151.13 0)
@@
 			)
 		)
-		(property "Footprint" "Capacitor_SMD:C_0603_1608Metric"
+		(property "Footprint" "Capacitor_SMD:C_0805_2012Metric"
 			(at 200.66 43.18 0)
 			(hide yes)
@@
 			)
 		)
-		(property "Value" "47uF"
+		(property "Value" "22uF"
 			(at 123.19 42.6338 0)
 			(show_name no)
@@
 	)
 	(symbol
+		(lib_id "Diode:SMAJ24CA")
+		(at 86.36 40.64 90)
+		(unit 1)
+		(body_style 1)
+		(exclude_from_sim no)
+		(in_bom yes)
+		(on_board yes)
+		(in_pos_files yes)
+		(dnp no)
+		(fields_autoplaced yes)
+		(property "Reference" "D1"
+			(at 88.9 39.3699 90)
+			(show_name no)
+			(do_not_autoplace no)
+			(effects
+				(font
+					(size 1.27 1.27)
+				)
+				(justify right)
+			)
+		)
+		(property "Value" "SMAJ24CA"
+			(at 88.9 41.9099 90)
+			(show_name no)
+			(do_not_autoplace no)
+			(effects
+				(font
+					(size 1.27 1.27)
+				)
+				(justify right)
+			)
+		)
+		(property "Footprint" "Diode_SMD:D_SMA"
+			(at 91.44 40.64 0)
+			(hide yes)
+			(show_name no)
+			(do_not_autoplace no)
+			(effects
+				(font
+					(size 1.27 1.27)
+				)
+			)
+		)
+		(property "Datasheet" "https://www.littelfuse.com/media?resourcetype=datasheets&itemid=75e32973-b177-4ee3-a0ff-cedaf1abdb93&filename=smaj-datasheet"
+			(at 86.36 40.64 0)
+			(hide yes)
+			(show_name no)
+			(do_not_autoplace no)
+			(effects
+				(font
+					(size 1.27 1.27)
+				)
+			)
+		)
+		(property "Description" "400W bidirectional Transient Voltage Suppressor, 24.0Vr, SMA(DO-214AC)"
+			(at 86.36 40.64 0)
+			(hide yes)
+			(show_name no)
+			(do_not_autoplace no)
+			(effects
+				(font
+					(size 1.27 1.27)
+				)
+			)
+		)
+		(property "LCSC" "C148223"
+			(at 86.36 40.64 90)
+			(hide yes)
+			(show_name no)
+			(do_not_autoplace no)
+			(effects
+				(font
+					(size 1.27 1.27)
+				)
+			)
+		)
+		(pin "2"
+		)
+		(pin "1"
+		)
+		(instances
+			(project "modbus-th-sensor"
+				(path "/0ebab830-f561-40b5-8ce2-2e04f313e8a8"
+					(reference "D1")
+					(unit 1)
+				)
+			)
+		)
+	)
+	(symbol
 		(lib_id "power:GND")
 		(at 248.92 139.7 270)
@@
 			)
 		)
-		(property "Value" "100K"
+		(property "Value" "470K"
 			(at 105.41 45.7199 0)
 			(show_name no)
@@
 			)
 		)
-		(property "LCSC" "C25803"
+		(property "LCSC" "C23178"
 			(at 102.87 44.45 0)
 			(hide yes)

Commit message: Replaced Q1 (AO3401A) with a Schottky Diode (SS210)
Parts:
- removed D2: 10V, Diode_SMD:D_SOD-123, symbol Device:D_Zener_Small
- removed Q1: AO3401A, Package_TO_SOT_SMD:SOT-23, symbol Transistor_FET:AO3401A
- removed R1: 470K, Resistor_SMD:R_0603_1608Metric, symbol Device:R_Small
- added D2: SS210, Diode_SMD:D_SMA, symbol Device:D_Schottky_Small
- renumbered R2 to R1, R3 to R2, R6 to R3
Connections:
- net at D1.2 (A2), F1.2: now also D2.2 (A)
- net at C1.1, C2.1, C3.1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: now also D2.1 (K)
Other:
- note removed: "Reverse Polarity Protection"
- moved on the sheet: R2

Commit message: Corrected C13 footprint
Parts:
- C13: footprint Capacitor_SMD:C_0603_1608Metric -> Capacitor_SMD:C_0402_1005Metric
Changed lines of the file:
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@@
 			)
 		)
-		(property "Footprint" "Capacitor_SMD:C_0603_1608Metric"
+		(property "Footprint" "Capacitor_SMD:C_0402_1005Metric"
 			(at 45.72 107.95 0)
 			(hide yes)

Commit message: Reversed FTDI connector so it is the right way round
Parts:
- R1: LCSC (none) -> C25804
- R2: value 330R -> 1K; LCSC (none) -> C21190
Connections:
- net +3.3V: now also J2.3 (Pin_3); no longer J2.4 (Pin_4)
- net GND: now also J2.1 (Pin_1), J2.2 (Pin_2); no longer J2.5 (Pin_5), J2.6 (Pin_6)
- net at C13.1: now also J2.6 (Pin_6); no longer J2.1 (Pin_1)
- net RXD renamed RXI
- net RXI: now also J2.4 (Pin_4); no longer J2.2 (Pin_2)
- net TXD renamed TXO
- net TXO: now also J2.5 (Pin_5); no longer J2.3 (Pin_3)
Other:
- moved on the sheet: C13, J2, R1

Commit message: Switched SMAJ24CA to a JLC basic part
Parts:
- D1: LCSC C148223 -> C19077542
Changed lines of the file:
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@@
 			)
 		)
-		(property "LCSC" "C148223"
+		(property "LCSC" "C19077542"
 			(at 86.36 40.64 90)
 			(hide yes)
