File: sht4x-breakout/sht4x-breakout.kicad_sch (KiCad schematic)
At the start: 5 parts, among them U1 SHT4x

Commit message: Added breakout PCB design
Connections:
- net +3.3V: now also J1.5 (Pin_5); no longer J1.1 (Pin_1)
- net GND: now also J1.1 (Pin_1); no longer J1.5 (Pin_5)
- net SDA: now also J1.4 (Pin_4); no longer J1.2 (Pin_2)
Changed lines of the file:
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@@
 		(lib_id "Connector_Generic:Conn_01x05")
 		(at 220.98 87.63 0)
+		(mirror x)
 		(unit 1)
 		(body_style 1)

Commit message: Breakout board revision 2: square outline and mounting hole - Changed the outline to a plain 19 x 19 mm square, removing the narrow header end - Added an M2.5 mounting hole (H1) at X 2.7, Y 2.7 to the schematic and PCB - J1 uses the vertical header footprint for cleaner silkscreen, with the right-angle 3D model - Set the board design rules to JLCPCB's manufacturing limits - Hid the PWR_FLAG values in the schematic
Parts:
- added H1: MountingHole, MountingHole:MountingHole_2.7mm_M2.5, symbol Mechanical:MountingHole
- J1: footprint Connector_PinHeader_2.54mm:PinHeader_1x05_P2.54mm_Horizontal -> Connector_PinHeader_2.54mm:PinHeader_1x05_P2.54mm_Vertical
Changed lines of the file:
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@@
 	(title_block
 		(title "SHT41 Breakout Module")
-		(date "2026-10-08")
-		(rev "1")
+		(date "2026-10-18")
+		(rev "2")
 		(company "aelius labs")
 	)
@@
 			)
 		)
-		(property "Footprint" "Connector_PinHeader_2.54mm:PinHeader_1x05_P2.54mm_Horizontal"
+		(property "Footprint" "Connector_PinHeader_2.54mm:PinHeader_1x05_P2.54mm_Vertical"
 			(at 220.98 87.63 0)
 			(hide yes)
@@
 		(property "Value" "PWR_FLAG"
 			(at 205.74 96.52 0)
+			(hide yes)
 			(show_name no)
 			(do_not_autoplace no)
@@
 	)
 	(symbol
+		(lib_id "Mechanical:MountingHole")
+		(at 220.98 106.68 0)
+		(unit 1)
+		(body_style 1)
+		(exclude_from_sim no)
+		(in_bom no)
+		(on_board yes)
+		(in_pos_files yes)
+		(dnp no)
+		(fields_autoplaced yes)
+		(property "Reference" "H1"
+			(at 223.52 105.41 0)
+			(show_name no)
+			(do_not_autoplace no)
+			(effects
+				(font
+					(size 1.27 1.27)
+				)
+				(justify left)
+			)
+		)
+		(property "Value" "MountingHole"
+			(at 223.52 107.95 0)
+			(show_name no)
+			(do_not_autoplace no)
+			(effects
+				(font
+					(size 1.27 1.27)
+				)
+				(justify left)
+			)
+		)
+		(property "Footprint" "MountingHole:MountingHole_2.7mm_M2.5"
+			(at 220.98 106.68 0)
+			(hide yes)
+			(show_name no)
+			(do_not_autoplace no)
+			(effects
+				(font
+					(size 1.27 1.27)
+				)
+			)
+		)
+		(property "Datasheet" ""
+			(at 220.98 106.68 0)
+			(hide yes)
+			(show_name no)
+			(do_not_autoplace no)
+			(effects
+				(font
+					(size 1.27 1.27)
+				)
+			)
+		)
+		(property "Description" "Mounting Hole without connection"
+			(at 220.98 106.68 0)
+			(hide yes)
+			(show_name no)
+			(do_not_autoplace no)
+			(effects
+				(font
+					(size 1.27 1.27)
+				)
+			)
+		)
+		(instances
+			(project "sht4x-breakout"
+				(path "/740cdee0-8bf3-45f0-a93f-324941fef48d"
+					(reference "H1")
+					(unit 1)
+				)
+			)
+		)
+	)
+	(symbol
 		(lib_id "power:+3.3V")
 		(at 198.12 80.01 0)
@@
 		(property "Value" "PWR_FLAG"
 			(at 205.74 78.74 0)
-			(show_name no)
-			(do_not_autoplace no)
+			(hide yes)
+			(show_name no)
+			(do_not_autoplace no)

Commit message: Minor adjustments and label changes
Parts:
- J1: value (none) -> 1x5 R/A header
- U1: value SHT4x -> SHT41-AD1B-R2
Changed lines of the file:
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@@
 			)
 		)
-		(property "Value" ""
+		(property "Value" "1x5 R/A header"
 			(at 220.98 95.25 0)
 			(show_name no)
@@
 		(dnp no)
 		(property "Reference" "U1"
-			(at 132.334 77.216 0)
-			(show_name no)
-			(do_not_autoplace no)
-			(effects
-				(font
-					(size 1.27 1.27)
-				)
-				(justify left)
-			)
-		)
-		(property "Value" "SHT4x"
-			(at 132.08 79.756 0)
-			(show_name no)
-			(do_not_autoplace no)
-			(effects
-				(font
-					(size 1.27 1.27)
-				)
-				(justify left)
-			)
-		)
+			(at 139.7 97.79 0)
+			(show_name no)
+			(do_not_autoplace no)
+			(effects
+				(font
+					(size 1.27 1.27)
+				)
+				(justify right)
+			)
+		)
+		(property "Value" "SHT41-AD1B-R2"
+			(at 139.7 100.33 0)
+			(show_name no)
+			(do_not_autoplace no)
+			(effects
+				(font
+					(size 1.27 1.27)
+				)
+				(justify right)
+			)
+		)
